File: pcb/v3.0/main/a4988.kicad_sch (KiCad schematic)
At the start: 5 parts, among them J4 Conn_01x04_Female, U4 a4988

Commit message: feat: update schematic
Parts:
- added D10: LED4, LED_SMD:LED_0603_1608Metric, symbol Device:LED
- added R36: 1k, Resistor_SMD:R_0603_1608Metric_Pad0.98x0.95mm_HandSolder, symbol Device:R_Small
- J4: value Conn_01x04_Female -> XH
- R5, R6: footprint Resistor_SMD:R_0805_2012Metric_Pad1.20x1.40mm_HandSolder -> Resistor_SMD:R_0603_1608Metric
Connections:
- net ENBLE: now also R36.1
- net GND: now also D10.1 (K)
- new net: D10.2 (A), R36.2
Other:
- moved on the sheet: R6

Commit message: feat: parts alignment (wip)
Parts:
- removed R5: 10k, Resistor_SMD:R_0603_1608Metric, symbol Device:R_Small
- J5: renamed from J4; footprint Connector_PinSocket_2.54mm:PinSocket_1x04_P2.54mm_Horizontal -> Connector_JST:JST_XH_B4B-XH-A_1x04_P2.50mm_Vertical
- renumbered C3 to C18, D10 to D11, R36 to R18, R6 to R19, U4 to U7
