File: pcb/v3.0/main/led.kicad_sch (KiCad schematic)
At the start: 5 parts, among them J8 Conn_01x02_Female, Q2 BSS138

Commit message: feat: update schematic
Parts:
- removed RV2: R_Potentiometer_Small, Potentiometer_THT:Potentiometer_Vishay_T73YP_Vertical, symbol Device:R_Potentiometer_Small
- J8: value Conn_01x02_Female -> PH; footprint Connector_PinSocket_2.54mm:PinSocket_1x02_P2.54mm_Horizontal -> Connector_JST:JST_PH_S2B-PH-K_1x02_P2.00mm_Horizontal
Connections:
- net GND: now also Q2.2 (S), R14.2; no longer J8.2 (Pin_2)
- net +BATT: no longer names the net of Q2.3 (D)
- net +BATT: now also J8.2 (Pin_2)
- new net VDD: J8.1 (Pin_1)
Other:
- moved on the sheet: J8, Q2, R13, R14

Commit message: feat: parts alignment (wip)
Parts:
- renumbered J8 to J9, Q2 to Q1, R13 to R26, R14 to R27
Changed lines of the file:
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@@
 		(on_board yes)
 		(dnp no)
-		(property "Reference" "Q2"
+		(property "Reference" "Q1"
 			(at 160.1216 90.2716 0)
 			(effects
@@
 		(on_board yes)
 		(dnp no)
-		(property "Reference" "R13"
+		(property "Reference" "R26"
 			(at 139.7 86.36 90)
 			(effects
@@
 			(project ""
 				(path "/1630ca0c-51c9-4aeb-9f5b-af64c3de63e1/74c6b7b8-a0c7-42ac-83d9-9103ac04caf3"
-					(reference "R11")
-					(unit 1)
-				)
-				(path "/1630ca0c-51c9-4aeb-9f5b-af64c3de63e1/921fc570-1318-4fd8-abfd-17fb575b4358"
-					(reference "R17")
-					(unit 1)
-				)
-				(path "/1630ca0c-51c9-4aeb-9f5b-af64c3de63e1/b78c16da-74af-4334-9017-c2140b9b5726"
-					(reference "R19")
-					(unit 1)
-				)
-				(path "/1630ca0c-51c9-4aeb-9f5b-af64c3de63e1/ded0eead-ed4f-4fa9-a2ac-ecfeb8f2a1bb"
-					(reference "R13")
+					(reference "R26")
+					(unit 1)
+				)
+				(path "/1630ca0c-51c9-4aeb-9f5b-af64c3de63e1/921fc570-1318-4fd8-abfd-17fb575b4358"
+					(reference "R32")
+					(unit 1)
+				)
+				(path "/1630ca0c-51c9-4aeb-9f5b-af64c3de63e1/b78c16da-74af-4334-9017-c2140b9b5726"
+					(reference "R34")
+					(unit 1)
+				)
+				(path "/1630ca0c-51c9-4aeb-9f5b-af64c3de63e1/ded0eead-ed4f-4fa9-a2ac-ecfeb8f2a1bb"
+					(reference "R28")
 					(unit 1)
 				)
@@
 		(dnp no)
 		(fields_autoplaced yes)
-		(property "Reference" "#PWR049"
+		(property "Reference" "#PWR0103"
 			(at 157.48 74.93 0)
 			(effects
@@
 			(project "main"
 				(path "/1630ca0c-51c9-4aeb-9f5b-af64c3de63e1/74c6b7b8-a0c7-42ac-83d9-9103ac04caf3"
-					(reference "#PWR049")
-					(unit 1)
-				)
-				(path "/1630ca0c-51c9-4aeb-9f5b-af64c3de63e1/921fc570-1318-4fd8-abfd-17fb575b4358"
-					(reference "#PWR062")
-					(unit 1)
-				)
-				(path "/1630ca0c-51c9-4aeb-9f5b-af64c3de63e1/b78c16da-74af-4334-9017-c2140b9b5726"
-					(reference "#PWR065")
-					(unit 1)
-				)
-				(path "/1630ca0c-51c9-4aeb-9f5b-af64c3de63e1/ded0eead-ed4f-4fa9-a2ac-ecfeb8f2a1bb"
-					(reference "#PWR052")
+					(reference "#PWR0103")
+					(unit 1)
+				)
+				(path "/1630ca0c-51c9-4aeb-9f5b-af64c3de63e1/921fc570-1318-4fd8-abfd-17fb575b4358"
+					(reference "#PWR0114")
+					(unit 1)
+				)
+				(path "/1630ca0c-51c9-4aeb-9f5b-af64c3de63e1/b78c16da-74af-4334-9017-c2140b9b5726"
+					(reference "#PWR0116")
+					(unit 1)
+				)
+				(path "/1630ca0c-51c9-4aeb-9f5b-af64c3de63e1/ded0eead-ed4f-4fa9-a2ac-ecfeb8f2a1bb"
+					(reference "#PWR0105")
 					(unit 1)
 				)
@@
 		(dnp no)
 		(fields_autoplaced yes)
-		(property "Reference" "J8"
+		(property "Reference" "J9"
 			(at 163.83 77.4699 0)
 			(effects
@@
 			(project ""
 				(path "/1630ca0c-51c9-4aeb-9f5b-af64c3de63e1/74c6b7b8-a0c7-42ac-83d9-9103ac04caf3"
-					(reference "J7")
-					(unit 1)
-				)
-				(path "/1630ca0c-51c9-4aeb-9f5b-af64c3de63e1/921fc570-1318-4fd8-abfd-17fb575b4358"
+					(reference "J9")
+					(unit 1)
+				)
+				(path "/1630ca0c-51c9-4aeb-9f5b-af64c3de63e1/921fc570-1318-4fd8-abfd-17fb575b4358"
+					(reference "J12")
+					(unit 1)
+				)
+				(path "/1630ca0c-51c9-4aeb-9f5b-af64c3de63e1/b78c16da-74af-4334-9017-c2140b9b5726"
+					(reference "J13")
+					(unit 1)
+				)
+				(path "/1630ca0c-51c9-4aeb-9f5b-af64c3de63e1/ded0eead-ed4f-4fa9-a2ac-ecfeb8f2a1bb"
 					(reference "J10")
-					(unit 1)
-				)
-				(path "/1630ca0c-51c9-4aeb-9f5b-af64c3de63e1/b78c16da-74af-4334-9017-c2140b9b5726"
-					(reference "J11")
-					(unit 1)
-				)
-				(path "/1630ca0c-51c9-4aeb-9f5b-af64c3de63e1/ded0eead-ed4f-4fa9-a2ac-ecfeb8f2a1bb"
-					(reference "J8")
 					(unit 1)
 				)
@@
 		(on_board yes)
 		(dnp no)
-		(property "Reference" "R14"
+		(property "Reference" "R27"
 			(at 150.0886 96.6216 0)
 			(effects
@@
 			(project ""
 				(path "/1630ca0c-51c9-4aeb-9f5b-af64c3de63e1/74c6b7b8-a0c7-42ac-83d9-9103ac04caf3"
-					(reference "R12")
-					(unit 1)
-				)
-				(path "/1630ca0c-51c9-4aeb-9f5b-af64c3de63e1/921fc570-1318-4fd8-abfd-17fb575b4358"
-					(reference "R18")
-					(unit 1)
-				)
-				(path "/1630ca0c-51c9-4aeb-9f5b-af64c3de63e1/b78c16da-74af-4334-9017-c2140b9b5726"
-					(reference "R20")
-					(unit 1)
-				)
-				(path "/1630ca0c-51c9-4aeb-9f5b-af64c3de63e1/ded0eead-ed4f-4fa9-a2ac-ecfeb8f2a1bb"
-					(reference "R14")
+					(reference "R27")
+					(unit 1)
+				)
+				(path "/1630ca0c-51c9-4aeb-9f5b-af64c3de63e1/921fc570-1318-4fd8-abfd-17fb575b4358"
+					(reference "R33")
+					(unit 1)
+				)
+				(path "/1630ca0c-51c9-4aeb-9f5b-af64c3de63e1/b78c16da-74af-4334-9017-c2140b9b5726"
+					(reference "R35")
+					(unit 1)
+				)
+				(path "/1630ca0c-51c9-4aeb-9f5b-af64c3de63e1/ded0eead-ed4f-4fa9-a2ac-ecfeb8f2a1bb"
+					(reference "R29")
 					(unit 1)
 				)
@@
 		(dnp no)
 		(fields_autoplaced yes)
-		(property "Reference" "#PWR051"
+		(property "Reference" "#PWR0104"
 			(at 157.48 113.03 0)
 			(effects
@@
 			(project ""
 				(path "/1630ca0c-51c9-4aeb-9f5b-af64c3de63e1/74c6b7b8-a0c7-42ac-83d9-9103ac04caf3"
-					(reference "#PWR048")
-					(unit 1)
-				)
-				(path "/1630ca0c-51c9-4aeb-9f5b-af64c3de63e1/921fc570-1318-4fd8-abfd-17fb575b4358"
-					(reference "#PWR061")
-					(unit 1)
-				)
-				(path "/1630ca0c-51c9-4aeb-9f5b-af64c3de63e1/b78c16da-74af-4334-9017-c2140b9b5726"
-					(reference "#PWR064")
-					(unit 1)
-				)
-				(path "/1630ca0c-51c9-4aeb-9f5b-af64c3de63e1/ded0eead-ed4f-4fa9-a2ac-ecfeb8f2a1bb"
-					(reference "#PWR051")
-					(unit 1)
-				)
+					(reference "#PWR0104")
+					(unit 1)
+				)
+				(path "/1630ca0c-51c9-4aeb-9f5b-af64c3de63e1/921fc570-1318-4fd8-abfd-17fb575b4358"
+					(reference "#PWR0115")
+					(unit 1)
+				)
+				(path "/1630ca0c-51c9-4aeb-9f5b-af64c3de63e1/b78c16da-74af-4334-9017-c2140b9b5726"
+					(reference "#PWR0117")
+					(unit 1)
+				)
+				(path "/1630ca0c-51c9-4aeb-9f5b-af64c3de63e1/ded0eead-ed4f-4fa9-a2ac-ecfeb8f2a1bb"
+					(reference "#PWR0106")
+					(unit 1)
+				)
