File: pcb/v3.0/main/power.kicad_sch (KiCad schematic)
At the start: 1 part, among them J1 Barrel_Jack

Commit message: feat: update schematic
Parts:
- added C10: 20u, Capacitor_SMD:C_0603_1608Metric_Pad1.08x0.95mm_HandSolder, symbol Device:C_Small
- added C11, C13: 1u, Capacitor_SMD:C_0603_1608Metric_Pad1.08x0.95mm_HandSolder, symbol Device:C_Small
- added C12: 0.01u, Capacitor_SMD:C_0603_1608Metric_Pad1.08x0.95mm_HandSolder, symbol Device:C_Small
- added C7: 100u, Capacitor_THT:CP_Radial_D10.0mm_P5.00mm, symbol Device:C_Polarized
- added C8, C9: 0.1u, Capacitor_SMD:C_0603_1608Metric_Pad1.08x0.95mm_HandSolder, symbol Device:C_Small
- added D1, D2, D3: LED, LED_SMD:LED_0603_1608Metric, symbol Device:LED
- added F1: 1A, Fuse:Fuseholder_Clip-5x20mm_Eaton_1A5601-01_Inline_P20.80x6.76mm_D1.70mm_Horizontal, symbol Device:Fuse_Small
- added R21: 20k, Resistor_SMD:R_0603_1608Metric_Pad0.98x0.95mm_HandSolder, symbol Device:R_Small
- added R22: 1.8k, Resistor_SMD:R_0603_1608Metric_Pad0.98x0.95mm_HandSolder, symbol Device:R_Small
- added R23: 1k, Resistor_SMD:R_0603_1608Metric_Pad0.98x0.95mm_HandSolder, symbol Device:R_Small
- added R24: 133, Resistor_SMD:R_1206_3216Metric_Pad1.30x1.75mm_HandSolder, symbol Device:R_Small
- added U8: LXDC55FAAA-203, My_Device:LXDC55FAAA-203, symbol My_Device:LXDC55FAAA-203
- added U9: NJM12877F33-TE1, Package_TO_SOT_SMD:SOT-23-5_HandSoldering, symbol bldc_lib:NJM12877F33-TE1
Connections:
- net +BATT: now also C7.1, F1.1
- net GND: now also C10.2, C11.2, C12.2, C13.2, C7.2, C8.2, C9.2, D1.1 (K), D2.1 (K), D3.1 (K), R24.2, U8.12 (GND), U8.13 (GND), U8.14 (GND), U8.6 (GND), U9.2 (GND)
- new net: C12.1, U9.4 (Cs)
- new net: D3.2 (A), R23.2
- new net: R24.1, U8.11 (FB)
- new net: D1.2 (A), R21.2
- new net: D2.2 (A), R22.2
- new net +3.3V: C13.1, U9.5 (VOUT)
- new net +3V3: R23.1
- new net +5V: C10.1, C11.1, C9.1, R22.1, U8.7 (VOUT), U8.8 (VOUT), U8.9 (VOUT), U9.1 (VIN), U9.3 (CONTROL)
- new net VDD: C8.1, F1.2, R21.1, U8.1 (EN), U8.3 (VIN), U8.4 (VIN), U8.5 (VIN)
Other:
- note added: "Blue"
- moved on the sheet: J1

Commit message: feat: parts alignment (wip)
Parts:
- F1: footprint Fuse:Fuseholder_Clip-5x20mm_Eaton_1A5601-01_Inline_P20.80x6.76mm_D1.70mm_Horizontal -> Fuse:Fuse_1206_3216Metric
- renumbered C7 to C10, C8 to C11, C9 to C12, C10 to C13, C11 to C14, C12 to C15, C13 to C16, D1 to D7, D2 to D8, D3 to D9, J1 to J3, R24 to R12, R21 to R13, R22 to R14, R23 to R15, U8 to U4, U9 to U5

Commit message: feat: finish pcb design
Parts:
- U4: footprint My_Device:LXDC55FAAA-203 -> mylib:LXDC55FAAA203
Connections:
- net +3V3 is gone; now on net +3.3V: R15.1
- net GND: now also R13.2; no longer D7.1 (K)
- net VDD: now also D7.2 (A); no longer R13.1
- new net: D7.1 (K), R13.1
Other:
- moved on the sheet: D7, R13
Changed lines of the file:
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@@
 	(wire
 		(pts
-			(xy 234.95 96.52) (xy 234.95 90.17)
-		)
-		(stroke
-			(width 0)
-			(type default)
-		)
-	)
-	(wire
-		(pts
 			(xy 44.45 114.3) (xy 50.8 114.3)
 		)
@@
 	(wire
 		(pts
+			(xy 234.95 111.76) (xy 234.95 115.57)
+		)
+		(stroke
+			(width 0)
+			(type default)
+		)
+	)
+	(wire
+		(pts
 			(xy 102.87 100.33) (xy 97.79 100.33)
 		)
@@
 	(wire
 		(pts
-			(xy 59.69 95.25) (xy 59.69 100.33)
+			(xy 234.95 102.87) (xy 234.95 106.68)
 		)
 		(stroke
@@
 	(wire
 		(pts
-			(xy 246.38 111.76) (xy 246.38 115.57)
+			(xy 59.69 95.25) (xy 59.69 100.33)
 		)
 		(stroke
@@
 	(wire
 		(pts
-			(xy 77.47 95.25) (xy 71.12 95.25)
+			(xy 234.95 90.17) (xy 234.95 95.25)
 		)
 		(stroke
@@
 	(wire
 		(pts
-			(xy 116.84 113.03) (xy 114.3 113.03)
+			(xy 246.38 111.76) (xy 246.38 115.57)
 		)
 		(stroke
@@
 	(wire
 		(pts
-			(xy 92.71 104.14) (xy 92.71 95.25)
+			(xy 77.47 95.25) (xy 71.12 95.25)
 		)
 		(stroke
@@
 	(wire
 		(pts
-			(xy 135.89 100.33) (xy 135.89 97.79)
+			(xy 116.84 113.03) (xy 114.3 113.03)
 		)
 		(stroke
@@
 	(wire
 		(pts
-			(xy 171.45 102.87) (xy 171.45 100.33)
+			(xy 92.71 104.14) (xy 92.71 95.25)
 		)
 		(stroke
@@
 	(wire
 		(pts
-			(xy 163.83 110.49) (xy 163.83 115.57)
+			(xy 135.89 100.33) (xy 135.89 97.79)
 		)
 		(stroke
@@
 	(wire
 		(pts
-			(xy 59.69 95.25) (xy 59.69 90.17)
+			(xy 171.45 102.87) (xy 171.45 100.33)
 		)
 		(stroke
@@
 	(wire
 		(pts
-			(xy 135.89 97.79) (xy 135.89 95.25)
+			(xy 163.83 110.49) (xy 163.83 115.57)
 		)
 		(stroke
@@
 	(wire
 		(pts
-			(xy 50.8 95.25) (xy 59.69 95.25)
+			(xy 59.69 95.25) (xy 59.69 90.17)
 		)
 		(stroke
@@
 	(wire
 		(pts
-			(xy 147.32 115.57) (xy 147.32 109.22)
+			(xy 135.89 97.79) (xy 135.89 95.25)
 		)
 		(stroke
@@
 	(wire
 		(pts
-			(xy 175.26 105.41) (xy 171.45 105.41)
+			(xy 50.8 95.25) (xy 59.69 95.25)
 		)
 		(stroke
@@
 	(wire
 		(pts
-			(xy 102.87 95.25) (xy 97.79 95.25)
+			(xy 147.32 115.57) (xy 147.32 109.22)
 		)
 		(stroke
@@
 	(wire
 		(pts
-			(xy 209.55 100.33) (xy 209.55 91.44)
+			(xy 175.26 105.41) (xy 171.45 105.41)
 		)
 		(stroke
@@
 	(wire
 		(pts
-			(xy 234.95 104.14) (xy 234.95 101.6)
+			(xy 102.87 95.25) (xy 97.79 95.25)
 		)
 		(stroke
@@
 	(wire
 		(pts
-			(xy 234.95 111.76) (xy 234.95 115.57)
+			(xy 209.55 100.33) (xy 209.55 91.44)
 		)
 		(stroke
@@
 			)
 		)
-		(property "Footprint" "My_Device:LXDC55FAAA-203"
+		(property "Footprint" "mylib:LXDC55FAAA203"
 			(at 109.22 91.44 0)
 			(effects
@@
 	(symbol
 		(lib_id "Device:R_Small")
-		(at 234.95 99.06 0)
+		(at 234.95 109.22 0)
 		(unit 1)
 		(exclude_from_sim no)
@@
 		(dnp no)
 		(property "Reference" "R13"
-			(at 236.4486 97.8916 0)
+			(at 236.4486 108.0516 0)
 			(effects
 				(font
@@
 		)
 		(property "Value" "20k"
-			(at 236.4486 100.203 0)
+			(at 236.4486 110.363 0)
 			(effects
 				(font
@@
 		)
 		(property "Footprint" "Resistor_SMD:R_0603_1608Metric_Pad0.98x0.95mm_HandSolder"
-			(at 234.95 99.06 0)
+			(at 234.95 109.22 0)
 			(effects
 				(font
@@
 		)
 		(property "Datasheet" "~"
-			(at 234.95 99.06 0)
+			(at 234.95 109.22 0)
 			(effects
 				(font
@@
 		)
 		(property "Description" ""
-			(at 234.95 99.06 0)
+			(at 234.95 109.22 0)
 			(effects
 				(font
@@
 	)
 	(symbol
+		(lib_id "power:+3.3V")
+		(at 257.81 90.17 0)
+		(unit 1)
+		(exclude_from_sim no)
+		(in_bom yes)
+		(on_board yes)
+		(dnp no)
+		(property "Reference" "#PWR066"
+			(at 257.81 93.98 0)
+			(effects
+				(font
+					(size 1.27 1.27)
+				)
+				(hide yes)
+			)
+		)
+		(property "Value" "+3.3V"
+			(at 257.81 85.09 0)
+			(effects
+				(font
+					(size 1.27 1.27)
+				)
+			)
+		)
+		(property "Footprint" ""
+			(at 257.81 90.17 0)
+			(effects
+				(font
+					(size 1.27 1.27)
+				)
+				(hide yes)
+			)
+		)
+		(property "Datasheet" ""
+			(at 257.81 90.17 0)
+			(effects
+				(font
+					(size 1.27 1.27)
+				)
+				(hide yes)
+			)
+		)
+		(property "Description" ""
+			(at 257.81 90.17 0)
+			(effects
+				(font
+					(size 1.27 1.27)
+				)
+				(hide yes)
+			)
+		)
+		(pin "1"
+		)
+		(instances
+			(project "main"
+				(path "/1630ca0c-51c9-4aeb-9f5b-af64c3de63e1/ff32423c-492c-45a2-9d86-d0144faa09a1"
+					(reference "#PWR066")
+					(unit 1)
+				)
+			)
+		)
+	)
+	(symbol
 		(lib_id "Device:R_Small")
 		(at 246.38 99.06 0)
@@
 	(symbol
 		(lib_id "Device:LED")
-		(at 234.95 107.95 270)
+		(at 234.95 99.06 270)
 		(mirror x)
 		(unit 1)
@@
 		(dnp no)
 		(property "Reference" "D7"
-			(at 236.982 106.9594 90)
+			(at 236.982 98.0694 90)
 			(effects
 				(font
@@
 		)
 		(property "Value" "LED"
-			(at 236.982 109.2708 90)
+			(at 236.982 100.3808 90)
 			(effects
 				(font
@@
 		)
 		(property "Footprint" "LED_SMD:LED_0603_1608Metric"
-			(at 234.95 107.95 0)
+			(at 234.95 99.06 0)
 			(effects
 				(font
@@
 		)
 		(property "Datasheet" "~"
-			(at 234.95 107.95 0)
+			(at 234.95 99.06 0)
 			(effects
 				(font
@@
 		)
 		(property "Description" ""
-			(at 234.95 107.95 0)
+			(at 234.95 99.06 0)
 			(effects
 				(font
@@
 					(unit 1)
 				)
-			)
-		)
-	)
-	(symbol
-		(lib_id "JXC_Control_Board-rescue:+3.3V-power")
-		(at 257.81 90.17 0)
-		(unit 1)
-		(exclude_from_sim no)
-		(in_bom yes)
-		(on_board yes)
-		(dnp no)
-		(property "Reference" "#PWR066"
-			(at 257.81 93.98 0)
-			(effects
-				(font
-					(size 1.27 1.27)
-				)
-				(hide yes)
-			)
-		)
-		(property "Value" "+3V3"
-			(at 258.191 85.7758 0)
-			(effects
-				(font
-					(size 1.27 1.27)
-				)
-			)
-		)
-		(property "Footprint" ""
-			(at 257.81 90.17 0)
-			(effects
-				(font
-					(size 1.27 1.27)
-				)
-				(hide yes)
-			)
-		)
-		(property "Datasheet" ""
-			(at 257.81 90.17 0)
-			(effects
-				(font
-					(size 1.27 1.27)
-				)
-				(hide yes)
-			)
-		)
-		(property "Description" ""
-			(at 257.81 90.17 0)
-			(effects
-				(font
-					(size 1.27 1.27)
-				)
-				(hide yes)
-			)
-		)
-		(pin "1"
-		)
-		(instances
-			(project "main"
-				(path "/1630ca0c-51c9-4aeb-9f5b-af64c3de63e1/ff32423c-492c-45a2-9d86-d0144faa09a1"
-					(reference "#PWR066")
-					(unit 1)
-				)
