File: pcb/v3.0/main/MicroController.kicad_sch (KiCad schematic)
At the start: 1 part, among them U1 RaspberryPi4

Commit message: feat: update schematic
Parts:
- added C14, C20, C21, C22, C23: 0.1u, Capacitor_SMD:C_0603_1608Metric, symbol Device:C_Small
- added C15, C16: 0.1u, Capacitor_SMD:C_0603_1608Metric_Pad1.08x0.95mm_HandSolder, symbol Device:C_Small
- added C17, C18: 10p, Capacitor_SMD:C_0402_1005Metric_Pad0.74x0.62mm_HandSolder, symbol Device:C_Small
- added C19: 4.7u, Capacitor_SMD:C_0603_1608Metric, symbol Device:C_Small
- added D4: LED5, LED_SMD:LED_0603_1608Metric, symbol Device:LED
- added D5: LED6, LED_SMD:LED_0603_1608Metric, symbol Device:LED
- added D6: LED1, LED_SMD:LED_0603_1608Metric, symbol Device:LED
- added D7: LED2, LED_SMD:LED_0603_1608Metric, symbol Device:LED
- added D8: LED3, LED_SMD:LED_0603_1608Metric, symbol Device:LED
- added D9: LED4, LED_SMD:LED_0603_1608Metric, symbol Device:LED
- added J12: PH, Connector_JST:JST_PH_S3B-PH-K_1x03_P2.00mm_Horizontal, symbol Connector:Conn_01x03_Socket
- added J13: Magnet, Connector_PinSocket_2.54mm:PinSocket_1x04_P2.54mm_Horizontal, symbol Connector:Conn_01x04_Female
- added R25: 120, Resistor_SMD:R_0603_1608Metric_Pad0.98x0.95mm_HandSolder, symbol Device:R_Small
- added R26, R27, R31, R32, R33, R34: 1k, Resistor_SMD:R_0603_1608Metric_Pad0.98x0.95mm_HandSolder, symbol Device:R_Small
- added R28, R30: 10k, Resistor_SMD:R_0603_1608Metric_Pad0.98x0.95mm_HandSolder, symbol Device:R_Small
- added R29: 1k, Resistor_SMD:R_0402_1005Metric_Pad0.72x0.64mm_HandSolder, symbol Device:R_Small
- added R35: 3.3k, Resistor_SMD:R_0603_1608Metric_Pad0.98x0.95mm_HandSolder, symbol Device:R_Small
- added RV5: 3.3k, Potentiometer_THT:Potentiometer_Vishay_T73YP_Vertical, symbol Device:R_Potentiometer_Small
- added SW1: RESET, half_mouse_lib:TVAF06-A020B-R, symbol My_Device:SKRPACE
- added SW2: USER, half_mouse_lib:TVAF06-A020B-R, symbol My_Device:SKRPACE
- added U10: MCP2562-E-SN, Package_SO:SOIC-8_3.9x4.9mm_P1.27mm, symbol Interface_CAN_LIN:MCP2562-E-SN
- added U11: STM32G431CB, Package_QFP:LQFP-48_7x7mm_P0.5mm, symbol bldc_lib:STM32G431CB
- added Y1: XRCGB16M000FXN02R0, mylib:XRCGB, symbol Device:Crystal_GND2_Small
Connections:
- net +3.3V: now also C19.1, C20.1, C21.1, C22.1, C23.1, R28.1, RV5.1, U11.1 (VBAT), U11.20 (VREF+), U11.21 (VDDA), U11.24 (VDD), U11.36 (VDD), U11.48 (VDD)
- net GND: now also C14.2, C15.2, C16.2, C17.2, C18.2, C19.2, C20.2, C21.2, C22.2, C23.2, D6.1 (K), D7.1 (K), D8.1 (K), D9.1 (K), J12.3 (Pin_3), J13.4 (Pin_4), R26.2, R27.2, R30.2, R35.2, SW1.2, SW2.1, U10.2 (VSS), U10.8 (STBY), U11.19 (VSSA), U11.23 (VSS), U11.35 (VSS), U11.47 (VSS), Y1.2
- new net: C17.1, R29.2, Y1.1
- new net: R30.1, U11.45 (PB8-BOOT0)
- new net: D7.2 (A), R32.2
- new net: D4.1 (K), R26.1
- new net: D5.1 (K), R27.1
- new net: D6.2 (A), R31.2
- new net: R35.1, RV5.3
- new net: D8.2 (A), R33.2
- new net: D9.2 (A), R34.2
- new net +5V: C14.1, U10.3 (VDD), U10.5 (Vio)
- new net CAN_H: J12.2 (Pin_2), R25.1, U10.7 (CANH)
- new net CAN_L: J12.1 (Pin_1), R25.2, U10.6 (CANL)
- new net CAN_RX: U10.4 (RXD), U11.33 (PA11)
- new net CAN_TX: U10.1 (TXD), U11.34 (PA12)
- new net LED1: R31.1, U11.22 (PB10)
- new net LED2: R32.1
- new net LED3: R33.1
- new net LED4: R34.1
- new net LED_CAN_RX: D5.2 (A), U11.32 (PA10)
- new net LED_CAN_TX: D4.2 (A), U11.31 (PA9)
- new net NRST: C15.1, J13.1 (Pin_1), SW1.1, U11.7 (PG10-NRST)
- new net OSC_IN: R29.1, U11.5 (PF0-OSC_IN)
- new net OSC_OUT: C18.1, U11.6 (PF0-OSC_OUT), Y1.3
- new net SW1: C16.1, R28.2, SW2.2, U11.30 (PA8)
- new net SWCLK: J13.2 (Pin_2), U11.38 (PA14)
- new net SWDIO: J13.3 (Pin_3), U11.37 (PA13)
- new net adc_speed: RV5.2
Other:
- note added: "CAN"
- note added: "Debug"
- note added: "HSE CLK"
- note added: "MCU"
- note added: "VDD"
- note added: "VDDA"
- note added: "Vref"
- moved on the sheet: U1

Commit message: feat: parts alignment (wip)
Parts:
- removed C23: 0.1u, Capacitor_SMD:C_0603_1608Metric, symbol Device:C_Small
- U1: footprint Connector_PinHeader_2.54mm:PinHeader_2x20_P2.54mm_Vertical -> (none)
- renumbered C17 to C1, C18 to C2, C15 to C3, C19 to C4, C20 to C5, C21 to C6, C16 to C7, C22 to C8, C14 to C9, D6 to D1, D7 to D2, D8 to D3, D9 to D4, D4 to D5, D5 to D6, J13 to J1, J12 to J2, R31 to R1, R26 to R10, R27 to R11, R29 to R2, R32 to R3, R33 to R4, R34 to R5, R30 to R6, R28 to R7, R35 to R8, R25 to R9, RV5 to RV1, U11 to U2, U10 to U3

Commit message: feat: finish pcb design
Parts:
- removed U1: RaspberryPi4, symbol stepper_music_lib:RaspberryPi4
- J1: footprint Connector_PinSocket_2.54mm:PinSocket_1x04_P2.54mm_Horizontal -> Connector_PinSocket_2.54mm:PinSocket_1x04_P2.54mm_Vertical
- Y1: footprint mylib:XRCGB -> bldc_lib:XRCGB
Connections:
- net DIR_B: now also U2.28 (PB14)
- net DIR_D: now also U2.27 (PB13)
- net DIR_F: now also U2.30 (PA8)
- net DIR_L: now also U2.14 (PA6)
- net DIR_R: now also U2.9 (PA1)
- net DIR_U: now also U2.15 (PA7)
- net ENABLE_B: now also U2.43 (PB6)
- net ENABLE_D: now also U2.46 (PB9)
- net ENABLE_F: now also U2.44 (PB7)
- net ENABLE_L: now also U2.4 (PC15)
- net ENABLE_R: now also U2.3 (PC14)
- net ENABLE_U: now also U2.2 (PC13)
- net LED1: now also U2.16 (PB0); no longer U2.22 (PB10)
- net LED2: now also U2.17 (PB1)
- net LED3: now also U2.18 (PB2)
- net LED4: now also U2.22 (PB10)
- net LED_B: now also U2.40 (PB3)
- net LED_CAN_RX: now also U2.26 (PB12); no longer U2.32 (PA10)
- net LED_CAN_TX: now also U2.25 (PB11); no longer U2.31 (PA9)
- net LED_F: now also U2.42 (PB5)
- net LED_L: now also U2.39 (PA15)
- net LED_R: now also U2.41 (PB4)
- net MS1: now also U2.10 (PA2)
- net MS2: now also U2.11 (PA3)
- net MS3: now also U2.13 (PA5)
- net STEP1: now also U2.29 (PB15)
- net SW1: now also U2.8 (PA0); no longer U2.30 (PA8)
- net SWCLK: now also J1.3 (Pin_3); no longer J1.2 (Pin_2)
- net SWDIO: now also J1.2 (Pin_2); no longer J1.3 (Pin_3)
- net adc_speed: now also U2.12 (PA4)

Commit message: fix: add UART
Parts:
- added J14: PH, Connector_JST:JST_PH_S2B-PH-K_1x02_P2.00mm_Horizontal, symbol Connector:Conn_01x02_Socket
Connections:
- net USART_TX: now reaches U2.31 (PA9)
- net USART_TX: now also J14.1 (Pin_1)
- net USART_RX: now reaches U2.32 (PA10)
- net USART_RX: now also J14.2 (Pin_2)
Other:
- moved on the sheet: J1
Changed lines of the file:
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@@
 	(wire
 		(pts
+			(xy 139.7 157.48) (xy 151.13 157.48)
+		)
+		(stroke
+			(width 0)
+			(type default)
+		)
+	)
+	(wire
+		(pts
 			(xy 22.86 180.34) (xy 25.4 180.34)
 		)
@@
 	(wire
 		(pts
-			(xy 151.13 147.32) (xy 147.32 147.32)
+			(xy 151.13 138.43) (xy 147.32 138.43)
 		)
 		(stroke
@@
 	(wire
 		(pts
-			(xy 143.51 139.7) (xy 151.13 139.7)
+			(xy 143.51 130.81) (xy 151.13 130.81)
 		)
 		(stroke
@@
 	(wire
 		(pts
-			(xy 143.51 142.24) (xy 151.13 142.24)
+			(xy 143.51 133.35) (xy 151.13 133.35)
 		)
 		(stroke
@@
 	(wire
 		(pts
+			(xy 101.6 66.04) (xy 91.44 66.04)
+		)
+		(stroke
+			(width 0)
+			(type default)
+		)
+	)
+	(wire
+		(pts
 			(xy 21.59 55.88) (xy 33.02 55.88)
 		)
@@
 	(wire
 		(pts
-			(xy 143.51 144.78) (xy 151.13 144.78)
+			(xy 143.51 135.89) (xy 151.13 135.89)
 		)
 		(stroke
@@
 	(wire
 		(pts
-			(xy 147.32 147.32) (xy 147.32 151.13)
+			(xy 147.32 138.43) (xy 147.32 142.24)
 		)
 		(stroke
@@
 		)
 	)
+	(wire
+		(pts
+			(xy 101.6 68.58) (xy 91.44 68.58)
+		)
+		(stroke
+			(width 0)
+			(type default)
+		)
+	)
 	(polyline
 		(pts
@@
 	(wire
 		(pts
+			(xy 139.7 154.94) (xy 151.13 154.94)
+		)
+		(stroke
+			(width 0)
+			(type default)
+		)
+	)
+	(wire
+		(pts
 			(xy 34.29 129.54) (xy 34.29 139.7)
 		)
@@
 		)
 	)
+	(label "USART_RX"
+		(at 101.6 66.04 180)
+		(fields_autoplaced yes)
+		(effects
+			(font
+				(size 1.27 1.27)
+			)
+			(justify right bottom)
+		)
+	)
+	(label "USART_TX"
+		(at 139.7 154.94 0)
+		(fields_autoplaced yes)
+		(effects
+			(font
+				(size 1.27 1.27)
+			)
+			(justify left bottom)
+		)
+	)
 	(label "LED4"
 		(at 53.34 129.54 270)
@@
 	)
 	(label "NRST"
-		(at 143.51 139.7 0)
+		(at 143.51 130.81 0)
 		(fields_autoplaced yes)
 		(effects
@@
 	)
 	(label "SWCLK"
-		(at 143.51 144.78 0)
+		(at 143.51 135.89 0)
 		(fields_autoplaced yes)
 		(effects
@@
 	)
 	(label "SWDIO"
-		(at 143.51 142.24 0)
+		(at 143.51 133.35 0)
 		(fields_autoplaced yes)
 		(effects
@@
 		)
 	)
+	(label "USART_TX"
+		(at 101.6 68.58 180)
+		(fields_autoplaced yes)
+		(effects
+			(font
+				(size 1.27 1.27)
+			)
+			(justify right bottom)
+		)
+	)
 	(label "LED1"
 		(at 55.88 109.22 90)
@@
 		)
 	)
+	(label "USART_RX"
+		(at 139.7 157.48 0)
+		(fields_autoplaced yes)
+		(effects
+			(font
+				(size 1.27 1.27)
+			)
+			(justify left bottom)
+		)
+	)
 	(label "adc_speed"
 		(at 166.37 64.77 180)
@@
 	)
 	(symbol
+		(lib_id "Connector:Conn_01x02_Socket")
+		(at 156.21 154.94 0)
+		(unit 1)
+		(exclude_from_sim no)
+		(in_bom yes)
+		(on_board yes)
+		(dnp no)
+		(fields_autoplaced yes)
+		(property "Reference" "J14"
+			(at 157.48 154.9399 0)
+			(effects
+				(font
+					(size 1.27 1.27)
+				)
+				(justify left)
+			)
+		)
+		(property "Value" "PH"
+			(at 157.48 157.4799 0)
+			(effects
+				(font
+					(size 1.27 1.27)
+				)
+				(justify left)
+			)
+		)
+		(property "Footprint" "Connector_JST:JST_PH_S2B-PH-K_1x02_P2.00mm_Horizontal"
+			(at 156.21 154.94 0)
+			(effects
+				(font
+					(size 1.27 1.27)
+				)
+				(hide yes)
+			)
+		)
+		(property "Datasheet" "~"
+			(at 156.21 154.94 0)
+			(effects
+				(font
+					(size 1.27 1.27)
+				)
+				(hide yes)
+			)
+		)
+		(property "Description" "Generic connector, single row, 01x02, script generated"
+			(at 156.21 154.94 0)
+			(effects
+				(font
+					(size 1.27 1.27)
+				)
+				(hide yes)
+			)
+		)
+		(pin "2"
+		)
+		(pin "1"
+		)
+		(instances
+			(project ""
+				(path "/1630ca0c-51c9-4aeb-9f5b-af64c3de63e1/890f87e9-49c3-4c63-bb8a-5b1e557cbd26"
+					(reference "J14")
+					(unit 1)
+				)
+			)
+		)
+	)
+	(symbol
 		(lib_id "power:+3.3V")
 		(at 76.2 99.06 180)
@@
 	(symbol
 		(lib_id "power:GND")
-		(at 147.32 151.13 0)
+		(at 147.32 142.24 0)
 		(unit 1)
 		(exclude_from_sim no)
@@
 		(fields_autoplaced yes)
 		(property "Reference" "#PWR035"
-			(at 147.32 157.48 0)
+			(at 147.32 148.59 0)
 			(effects
 				(font
@@
 		)
 		(property "Value" "GND"
-			(at 147.32 156.21 0)
+			(at 147.32 147.32 0)
 			(effects
 				(font
@@
 		)
 		(property "Footprint" ""
-			(at 147.32 151.13 0)
+			(at 147.32 142.24 0)
 			(effects
 				(font
@@
 		)
 		(property "Datasheet" ""
-			(at 147.32 151.13 0)
+			(at 147.32 142.24 0)
 			(effects
 				(font
@@
 		)
 		(property "Description" ""
-			(at 147.32 151.13 0)
+			(at 147.32 142.24 0)
 			(effects
 				(font
@@
 	(symbol
 		(lib_id "Connector:Conn_01x04_Female")
-		(at 156.21 142.24 0)
+		(at 156.21 133.35 0)
 		(unit 1)
 		(exclude_from_sim no)
@@
 		(fields_autoplaced yes)
 		(property "Reference" "J1"
-			(at 157.48 142.2399 0)
+			(at 157.48 133.3499 0)
 			(effects
 				(font
@@
 		)
 		(property "Value" "Magnet"
-			(at 157.48 144.7799 0)
+			(at 157.48 135.8899 0)
 			(effects
 				(font
@@
 		)
 		(property "Footprint" "Connector_PinSocket_2.54mm:PinSocket_1x04_P2.54mm_Vertical"
-			(at 156.21 142.24 0)
+			(at 156.21 133.35 0)
 			(effects
 				(font
@@
 		)
 		(property "Datasheet" "~"
-			(at 156.21 142.24 0)
+			(at 156.21 133.35 0)
 			(effects
 				(font
@@
 		)
 		(property "Description" ""
-			(at 156.21 142.24 0)
+			(at 156.21 133.35 0)
 			(effects
 				(font

Commit message: chore: add pdf
Parts:
- J14: footprint Connector_JST:JST_PH_S2B-PH-K_1x02_P2.00mm_Horizontal -> Connector_JST:JST_PH_S3B-PH-K_1x03_P2.00mm_Horizontal; symbol Connector:Conn_01x02_Socket -> Connector:Conn_01x03_Socket
Connections:
- net GND: now also J14.3 (Pin_3)
Other:
- moved on the sheet: J1
Changed lines of the file:
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@@
 	(wire
 		(pts
-			(xy 139.7 157.48) (xy 151.13 157.48)
-		)
-		(stroke
-			(width 0)
-			(type default)
-		)
-	)
-	(wire
-		(pts
 			(xy 22.86 180.34) (xy 25.4 180.34)
 		)
@@
 	(wire
 		(pts
-			(xy 151.13 138.43) (xy 147.32 138.43)
+			(xy 151.13 137.16) (xy 147.32 137.16)
 		)
 		(stroke
@@
 	(wire
 		(pts
-			(xy 143.51 130.81) (xy 151.13 130.81)
+			(xy 143.51 129.54) (xy 151.13 129.54)
 		)
 		(stroke
@@
 	(wire
 		(pts
-			(xy 143.51 133.35) (xy 151.13 133.35)
+			(xy 143.51 132.08) (xy 151.13 132.08)
 		)
 		(stroke
@@
 	(wire
 		(pts
+			(xy 147.32 156.21) (xy 151.13 156.21)
+		)
+		(stroke
+			(width 0)
+			(type default)
+		)
+	)
+	(wire
+		(pts
 			(xy 21.59 52.07) (xy 21.59 55.88)
 		)
@@
 	(wire
 		(pts
+			(xy 147.32 158.75) (xy 147.32 156.21)
+		)
+		(stroke
+			(width 0)
+			(type default)
+		)
+	)
+	(wire
+		(pts
 			(xy 92.71 143.51) (xy 90.17 143.51)
 		)
@@
 	(wire
 		(pts
-			(xy 143.51 135.89) (xy 151.13 135.89)
+			(xy 143.51 134.62) (xy 151.13 134.62)
 		)
 		(stroke
@@
 	(wire
 		(pts
-			(xy 147.32 138.43) (xy 147.32 142.24)
+			(xy 147.32 137.16) (xy 147.32 139.7)
 		)
 		(stroke
@@
 	(wire
 		(pts
-			(xy 91.44 81.28) (xy 104.14 81.28)
+			(xy 139.7 151.13) (xy 151.13 151.13)
 		)
 		(stroke
@@
 	(wire
 		(pts
-			(xy 217.17 107.95) (xy 217.17 109.22)
+			(xy 91.44 81.28) (xy 104.14 81.28)
 		)
 		(stroke
@@
 	(wire
 		(pts
-			(xy 139.7 154.94) (xy 151.13 154.94)
+			(xy 217.17 107.95) (xy 217.17 109.22)
 		)
 		(stroke
@@
 	(wire
 		(pts
+			(xy 139.7 153.67) (xy 151.13 153.67)
+		)
+		(stroke
+			(width 0)
+			(type default)
+		)
+	)
+	(wire
+		(pts
 			(xy 96.52 26.67) (xy 96.52 25.4)
 		)
@@
 	)
 	(label "USART_TX"
-		(at 139.7 154.94 0)
+		(at 139.7 151.13 0)
 		(fields_autoplaced yes)
 		(effects
@@
 	)
 	(label "NRST"
-		(at 143.51 130.81 0)
+		(at 143.51 129.54 0)
 		(fields_autoplaced yes)
 		(effects
@@
 	)
 	(label "SWCLK"
-		(at 143.51 135.89 0)
+		(at 143.51 134.62 0)
 		(fields_autoplaced yes)
 		(effects
@@
 	)
 	(label "SWDIO"
-		(at 143.51 133.35 0)
+		(at 143.51 132.08 0)
 		(fields_autoplaced yes)
 		(effects
@@
 	)
 	(label "USART_RX"
-		(at 139.7 157.48 0)
+		(at 139.7 153.67 0)
 		(fields_autoplaced yes)
 		(effects
@@
 	)
 	(symbol
-		(lib_id "Connector:Conn_01x02_Socket")
-		(at 156.21 154.94 0)
+		(lib_id "Connector:Conn_01x03_Socket")
+		(at 156.21 153.67 0)
 		(unit 1)
 		(exclude_from_sim no)
@@
 		(fields_autoplaced yes)
 		(property "Reference" "J14"
-			(at 157.48 154.9399 0)
+			(at 157.48 152.3999 0)
 			(effects
 				(font
@@
 		)
 		(property "Value" "PH"
-			(at 157.48 157.4799 0)
+			(at 157.48 154.9399 0)
 			(effects
 				(font
@@
 			)
 		)
-		(property "Footprint" "Connector_JST:JST_PH_S2B-PH-K_1x02_P2.00mm_Horizontal"
-			(at 156.21 154.94 0)
+		(property "Footprint" "Connector_JST:JST_PH_S3B-PH-K_1x03_P2.00mm_Horizontal"
+			(at 156.21 153.67 0)
 			(effects
 				(font
@@
 		)
 		(property "Datasheet" "~"
-			(at 156.21 154.94 0)
+			(at 156.21 153.67 0)
 			(effects
 				(font
@@
 			)
 		)
-		(property "Description" "Generic connector, single row, 01x02, script generated"
-			(at 156.21 154.94 0)
+		(property "Description" "Generic connector, single row, 01x03, script generated"
+			(at 156.21 153.67 0)
 			(effects
 				(font
@@
 		(pin "1"
 		)
+		(pin "3"
+		)
 		(instances
 			(project ""
@@
 	)
 	(symbol
+		(lib_id "power:GND")
+		(at 147.32 158.75 0)
+		(unit 1)
+		(exclude_from_sim no)
+		(in_bom yes)
+		(on_board yes)
+		(dnp no)
+		(fields_autoplaced yes)
+		(property "Reference" "#PWR01"
+			(at 147.32 165.1 0)
+			(effects
+				(font
+					(size 1.27 1.27)
+				)
+				(hide yes)
+			)
+		)
+		(property "Value" "GND"
+			(at 147.32 163.83 0)
+			(effects
+				(font
+					(size 1.27 1.27)
+				)
+			)
+		)
+		(property "Footprint" ""
+			(at 147.32 158.75 0)
+			(effects
+				(font
+					(size 1.27 1.27)
+				)
+				(hide yes)
+			)
+		)
+		(property "Datasheet" ""
+			(at 147.32 158.75 0)
+			(effects
+				(font
+					(size 1.27 1.27)
+				)
+				(hide yes)
+			)
+		)
+		(property "Description" ""
+			(at 147.32 158.75 0)
+			(effects
+				(font
+					(size 1.27 1.27)
+				)
+				(hide yes)
+			)
+		)
+		(pin "1"
+		)
+		(instances
+			(project "main"
+				(path "/1630ca0c-51c9-4aeb-9f5b-af64c3de63e1/890f87e9-49c3-4c63-bb8a-5b1e557cbd26"
+					(reference "#PWR01")
+					(unit 1)
+				)
+			)
+		)
+	)
+	(symbol
 		(lib_id "bldc_lib:STM32G431CB")
 		(at 62.23 69.85 0)
@@
 	(symbol
 		(lib_id "power:GND")
-		(at 147.32 142.24 0)
+		(at 147.32 139.7 0)
 		(unit 1)
 		(exclude_from_sim no)
@@
 		(fields_autoplaced yes)
 		(property "Reference" "#PWR035"
-			(at 147.32 148.59 0)
+			(at 147.32 146.05 0)
 			(effects
 				(font
@@
 		)
 		(property "Value" "GND"
-			(at 147.32 147.32 0)
+			(at 147.32 144.78 0)
 			(effects
 				(font
@@
 		)
 		(property "Footprint" ""
-			(at 147.32 142.24 0)
+			(at 147.32 139.7 0)
 			(effects
 				(font
@@
 		)
 		(property "Datasheet" ""
-			(at 147.32 142.24 0)
+			(at 147.32 139.7 0)
 			(effects
 				(font
@@
 		)
 		(property "Description" ""
-			(at 147.32 142.24 0)
+			(at 147.32 139.7 0)
 			(effects
 				(font
@@
 	(symbol
 		(lib_id "Connector:Conn_01x04_Female")
-		(at 156.21 133.35 0)
+		(at 156.21 132.08 0)
 		(unit 1)
 		(exclude_from_sim no)
@@
 		(fields_autoplaced yes)
 		(property "Reference" "J1"
-			(at 157.48 133.3499 0)
+			(at 157.48 132.0799 0)
 			(effects
 				(font
@@
 		)
 		(property "Value" "Magnet"
-			(at 157.48 135.8899 0)
+			(at 157.48 134.6199 0)
 			(effects
 				(font
@@
 		)
 		(property "Footprint" "Connector_PinSocket_2.54mm:PinSocket_1x04_P2.54mm_Vertical"
-			(at 156.21 133.35 0)
+			(at 156.21 132.08 0)
 			(effects
 				(font
@@
 		)
 		(property "Datasheet" "~"
-			(at 156.21 133.35 0)
+			(at 156.21 132.08 0)
 			(effects
 				(font
@@
 		)
 		(property "Description" ""
-			(at 156.21 133.35 0)
+			(at 156.21 132.08 0)
 			(effects
 				(font
