File: pcb/v3.0/main/main.kicad_pcb (KiCad board)
At the start: 2 copper layers, 95 x 72 mm, 52 parts, among them J1 Barrel_Jack, J10 Conn_01x02_Female, J11 Conn_01x02_Female, J2 Conn_01x04_Female, J3 Conn_01x04_Female, J4 Conn_01x04_Female, J5 Conn_01x04_Female, J6 Conn_01x04_Female, J7 Conn_01x02_Female, J8 Conn_01x02_Female, J9 Conn_01x04_Female, Q1 BSS138, Q2 BSS138, Q3 BSS138, Q4 BSS138, U1 RaspberryPi4, U2 a4988, U3 a4988, U4 a4988, U5 a4988, U6 a4988, U7 a4988

Commit message: feat: update schematic
Parts:
- removed RV1, RV2, RV3, RV4: R_Potentiometer_Small, Potentiometer_THT:Potentiometer_Vishay_T73YP_Vertical
- added C10: 20u, Capacitor_SMD:C_0603_1608Metric_Pad1.08x0.95mm_HandSolder, F.Cu at (43.6, 108.2)
- added C11: 1u, Capacitor_SMD:C_0603_1608Metric_Pad1.08x0.95mm_HandSolder, F.Cu at (43.6, 110.7)
- added C12: 0.01u, Capacitor_SMD:C_0603_1608Metric_Pad1.08x0.95mm_HandSolder, F.Cu at (43.6, 113.2)
- added C13: 1u, Capacitor_SMD:C_0603_1608Metric_Pad1.08x0.95mm_HandSolder, F.Cu at (43.6, 115.8)
- added C14: 0.1u, Capacitor_SMD:C_0603_1608Metric, F.Cu at (43.4, 86.1)
- added C15: 0.1u, Capacitor_SMD:C_0603_1608Metric_Pad1.08x0.95mm_HandSolder, F.Cu at (47.7, 82.8)
- added C16: 0.1u, Capacitor_SMD:C_0603_1608Metric_Pad1.08x0.95mm_HandSolder, F.Cu at (47.7, 85.4)
- added C17: 10p, Capacitor_SMD:C_0402_1005Metric_Pad0.74x0.62mm_HandSolder, F.Cu at (60.4, 78.4)
- added C18: 10p, Capacitor_SMD:C_0402_1005Metric_Pad0.74x0.62mm_HandSolder, F.Cu at (60.4, 80.3)
- added C19: 4.7u, Capacitor_SMD:C_0603_1608Metric, F.Cu at (43.4, 88.7)
- added C20: 0.1u, Capacitor_SMD:C_0603_1608Metric, F.Cu at (43.4, 91.2)
- added C21: 0.1u, Capacitor_SMD:C_0603_1608Metric, F.Cu at (43.4, 93.7)
- added C22: 0.1u, Capacitor_SMD:C_0603_1608Metric, F.Cu at (43.4, 96.2)
- added C23: 0.1u, Capacitor_SMD:C_0603_1608Metric, F.Cu at (43.4, 98.7)
- added C7: 100u, Capacitor_THT:CP_Radial_D10.0mm_P5.00mm, F.Cu at (49.3, 107.7)
- added C8: 0.1u, Capacitor_SMD:C_0603_1608Metric_Pad1.08x0.95mm_HandSolder, F.Cu at (43.6, 103.2)
- added C9: 0.1u, Capacitor_SMD:C_0603_1608Metric_Pad1.08x0.95mm_HandSolder, F.Cu at (43.6, 105.7)
- added D1: LED, LED_SMD:LED_0603_1608Metric, F.Cu at (59.6, 103.2)
- added D10: LED4, LED_SMD:LED_0603_1608Metric, F.Cu at (73.9, 87.3)
- added D11: LED4, LED_SMD:LED_0603_1608Metric, F.Cu at (74.9, 105.8)
- added D12: LED4, LED_SMD:LED_0603_1608Metric, F.Cu at (74.9, 120.0)
- added D13: LED4, LED_SMD:LED_0603_1608Metric, F.Cu at (73.9, 80.2)
- added D14: LED4, LED_SMD:LED_0603_1608Metric, F.Cu at (74.9, 112.8)
- added D15: LED4, LED_SMD:LED_0603_1608Metric, F.Cu at (73.9, 73.2)
- added D2: LED, LED_SMD:LED_0603_1608Metric, F.Cu at (59.6, 105.8)
- added D3: LED, LED_SMD:LED_0603_1608Metric, F.Cu at (59.6, 108.4)
- added D4: LED5, LED_SMD:LED_0603_1608Metric, F.Cu at (43.5, 70.6)
- added D5: LED6, LED_SMD:LED_0603_1608Metric, F.Cu at (43.5, 73.2)
- added D6: LED1, LED_SMD:LED_0603_1608Metric, F.Cu at (43.5, 75.8)
- added D7: LED2, LED_SMD:LED_0603_1608Metric, F.Cu at (43.5, 78.4)
- added D8: LED3, LED_SMD:LED_0603_1608Metric, F.Cu at (43.5, 81.0)
- added D9: LED4, LED_SMD:LED_0603_1608Metric, F.Cu at (43.5, 83.6)
- added F1: 1A, Fuse:Fuseholder_Clip-5x20mm_Eaton_1A5601-01_Inline_P20.80x6.76mm_D1.70mm_Horizontal, F.Cu at (47.9, 117.5)
- added J12: PH, Connector_JST:JST_PH_S3B-PH-K_1x03_P2.00mm_Horizontal, F.Cu at (100.7, 92.8)
- added J13: Magnet, Connector_PinSocket_2.54mm:PinSocket_1x04_P2.54mm_Horizontal, F.Cu at (56.6, 71.6)
- added R21: 20k, Resistor_SMD:R_0603_1608Metric_Pad0.98x0.95mm_HandSolder, F.Cu at (43.6, 118.3)
- added R22: 1.8k, Resistor_SMD:R_0603_1608Metric_Pad0.98x0.95mm_HandSolder, F.Cu at (43.6, 120.8)
- added R23: 1k, Resistor_SMD:R_0603_1608Metric_Pad0.98x0.95mm_HandSolder, F.Cu at (43.6, 123.3)
- added R24: 133, Resistor_SMD:R_1206_3216Metric_Pad1.30x1.75mm_HandSolder, F.Cu at (64.6, 108.4)
- added R25: 120, Resistor_SMD:R_0603_1608Metric_Pad0.98x0.95mm_HandSolder, F.Cu at (47.7, 87.9)
- added R26: 1k, Resistor_SMD:R_0603_1608Metric_Pad0.98x0.95mm_HandSolder, F.Cu at (47.7, 90.4)
- added R27: 1k, Resistor_SMD:R_0603_1608Metric_Pad0.98x0.95mm_HandSolder, F.Cu at (52.0, 82.8)
- added R28: 10k, Resistor_SMD:R_0603_1608Metric_Pad0.98x0.95mm_HandSolder, F.Cu at (52.0, 85.4)
- added R29: 1k, Resistor_SMD:R_0402_1005Metric_Pad0.72x0.64mm_HandSolder, F.Cu at (63.7, 78.4)
- added R30: 10k, Resistor_SMD:R_0603_1608Metric_Pad0.98x0.95mm_HandSolder, F.Cu at (52.0, 87.9)
- added R31: 1k, Resistor_SMD:R_0603_1608Metric_Pad0.98x0.95mm_HandSolder, F.Cu at (52.0, 90.4)
- added R32: 1k, Resistor_SMD:R_0603_1608Metric_Pad0.98x0.95mm_HandSolder, F.Cu at (56.4, 82.8)
- added R33: 1k, Resistor_SMD:R_0603_1608Metric_Pad0.98x0.95mm_HandSolder, F.Cu at (56.4, 85.4)
- added R34: 1k, Resistor_SMD:R_0603_1608Metric_Pad0.98x0.95mm_HandSolder, F.Cu at (56.4, 87.9)
- added R35: 3.3k, Resistor_SMD:R_0603_1608Metric_Pad0.98x0.95mm_HandSolder, F.Cu at (56.4, 90.4)
- added R36: 1k, Resistor_SMD:R_0603_1608Metric_Pad0.98x0.95mm_HandSolder, F.Cu at (74.1, 84.8)
- added R37: 1k, Resistor_SMD:R_0603_1608Metric_Pad0.98x0.95mm_HandSolder, F.Cu at (75.0, 103.2)
- added R38: 1k, Resistor_SMD:R_0603_1608Metric_Pad0.98x0.95mm_HandSolder, F.Cu at (75.0, 117.4)
- added R39: 1k, Resistor_SMD:R_0603_1608Metric_Pad0.98x0.95mm_HandSolder, F.Cu at (74.1, 77.7)
- added R40: 1k, Resistor_SMD:R_0603_1608Metric_Pad0.98x0.95mm_HandSolder, F.Cu at (75.0, 110.3)
- added R41: 1k, Resistor_SMD:R_0603_1608Metric_Pad0.98x0.95mm_HandSolder, F.Cu at (74.1, 70.6)
- added RV5: 3.3k, Potentiometer_THT:Potentiometer_Vishay_T73YP_Vertical, F.Cu at (49.9, 98.3)
- added SW1: RESET, half_mouse_lib:TVAF06-A020B-R, F.Cu at (62.1, 71.4)
- added SW2: USER, half_mouse_lib:TVAF06-A020B-R, F.Cu at (62.1, 75.4)
- added U10: MCP2562-E-SN, Package_SO:SOIC-8_3.9x4.9mm_P1.27mm, F.Cu at (62.8, 96.3)
- added U11: STM32G431CB, Package_QFP:LQFP-48_7x7mm_P0.5mm, F.Cu at (64.2, 87.3)
- added U9: NJM12877F33-TE1, Package_TO_SOT_SMD:SOT-23-5_HandSoldering, F.Cu at (64.6, 104.4)
- J10, J11, J7, J8: value Conn_01x02_Female -> PH; footprint Connector_PinSocket_2.54mm:PinSocket_1x02_P2.54mm_Horizontal -> Connector_JST:JST_PH_S2B-PH-K_1x02_P2.00mm_Horizontal
- J2, J3, J4, J5, J6, J9: value Conn_01x04_Female -> XH
- R1, R10, R15, R16, R2, R3, R4, R5, R6, R7, R8, R9: footprint Resistor_SMD:R_0805_2012Metric_Pad1.20x1.40mm_HandSolder -> Resistor_SMD:R_0603_1608Metric
- moved J8 13.1 mm to (100.7, 103.0), turned to -90 degrees
- moved J11 10.7 mm to (100.7, 110.0), turned to -90 degrees
- moved J10 1.99 mm to (100.7, 124.3), turned to -90 degrees
- moved J7 1.97 mm to (100.7, 117.2), turned to -90 degrees
Connections:
- J10 pad 1: Net-(Q3-Pad2) -> VDD
- J10 pad 2: GND -> Net-(J10-Pin_2)
- J11 pad 1: Net-(Q4-Pad2) -> VDD
- J11 pad 2: GND -> Net-(J11-Pin_2)
- J7 pad 1: Net-(Q1-Pad2) -> VDD
- J7 pad 2: GND -> Net-(J7-Pin_2)
- J8 pad 1: Net-(Q2-Pad2) -> VDD
- J8 pad 2: GND -> Net-(J8-Pin_2)
- Q1 pad 2: Net-(Q1-Pad2) -> GND
- Q1 pad 3: +BATT -> Net-(J7-Pin_2)
- Q2 pad 2: Net-(Q2-Pad2) -> GND
- Q2 pad 3: +BATT -> Net-(J8-Pin_2)
- Q3 pad 2: Net-(Q3-Pad2) -> GND
- Q3 pad 3: +BATT -> Net-(J10-Pin_2)
- Q4 pad 2: Net-(Q4-Pad2) -> GND
- Q4 pad 3: +BATT -> Net-(J11-Pin_2)
- R12 pad 2: Net-(Q1-Pad2) -> GND
- R14 pad 2: Net-(Q2-Pad2) -> GND
- R18 pad 2: Net-(Q3-Pad2) -> GND
- R20 pad 2: Net-(Q4-Pad2) -> GND
Routing:
- net +BATT: track 293.5 -> 254.7 mm
- net Net-(J11-Pin_2): track 0.00 -> 29.2 mm
- net Net-(Q4-Pad2): track 25.0 -> 0.00 mm
- net Net-(Q3-Pad2): track 24.0 -> 0.00 mm
- net GND: track 393.2 -> 410.6 mm
- net Net-(Q1-Pad2): track 15.1 -> 0.00 mm
- net Net-(Q2-Pad2): track 13.7 -> 0.00 mm
- net Net-(J8-Pin_2): track 0.00 -> 13.2 mm
- net (no net): track 0.00 -> 9.15 mm
- net VDD: track 0.00 -> 8.79 mm

Commit message: feat: parts alignment (wip)
Parts:
- removed C23: 0.1u, Capacitor_SMD:C_0603_1608Metric
- removed the R1 at (141.6, 88.0)
- removed the R15 at (135.0, 111.5)
- removed the R3 at (166.5, 88.1)
- removed the R5 at (117.6, 87.9)
- removed the R7 at (158.4, 111.4)
- removed the R9 at (182.2, 111.5)
- removed U1: RaspberryPi4, Connector_PinHeader_2.54mm:PinHeader_2x20_P2.54mm_Vertical
- F1: footprint Fuse:Fuseholder_Clip-5x20mm_Eaton_1A5601-01_Inline_P20.80x6.76mm_D1.70mm_Horizontal -> Fuse:Fuse_1206_3216Metric
- J11: renamed from J9; footprint Connector_PinSocket_2.54mm:PinSocket_1x04_P2.54mm_Horizontal -> Connector_JST:JST_XH_B4B-XH-A_1x04_P2.50mm_Vertical; moved to F.Cu
- J4: renamed from J2; footprint Connector_PinSocket_2.54mm:PinSocket_1x04_P2.54mm_Horizontal -> Connector_JST:JST_XH_B4B-XH-A_1x04_P2.50mm_Vertical; moved to F.Cu
- J5: renamed from J3; footprint Connector_PinSocket_2.54mm:PinSocket_1x04_P2.54mm_Horizontal -> Connector_JST:JST_XH_B4B-XH-A_1x04_P2.50mm_Vertical; moved to F.Cu
- J6: renamed from J4; footprint Connector_PinSocket_2.54mm:PinSocket_1x04_P2.54mm_Horizontal -> Connector_JST:JST_XH_B4B-XH-A_1x04_P2.50mm_Vertical; moved to F.Cu
- J7: renamed from J5; footprint Connector_PinSocket_2.54mm:PinSocket_1x04_P2.54mm_Horizontal -> Connector_JST:JST_XH_B4B-XH-A_1x04_P2.50mm_Vertical; moved to F.Cu
- J8: renamed from J6; footprint Connector_PinSocket_2.54mm:PinSocket_1x04_P2.54mm_Horizontal -> Connector_JST:JST_XH_B4B-XH-A_1x04_P2.50mm_Vertical; moved to F.Cu
- moved D15 105.6 mm to (179.2, 64.5)
- moved D10 105.2 mm to (179.1, 87.1)
- moved R30 105.1 mm to (179.0, 66.1)
- moved R16 105.0 mm to (179.0, 88.7)
- moved D14 104.2 mm to (179.1, 111.9)
- moved R24 104.0 mm to (179.0, 113.5)
- moved D12 97.5 mm to (155.0, 64.3)
- moved R20 95.0 mm to (154.9, 65.9)
- moved C11 92.2 mm to (117.1, 47.5)
- moved C12 92.2 mm to (117.1, 50.0)
- moved C13 92.2 mm to (117.1, 52.5)
- moved RV1 89.7 mm to (129.0, 55.9)
- moved C16 89.4 mm to (126.6, 82.4), turned to 90 degrees
- moved F1 88.7 mm to (123.0, 70.2), turned to 90 degrees
- moved R22 88.4 mm to (154.9, 113.5)
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- renumbered C17 to C1, C7 to C10, C8 to C11, C9 to C12, C10 to C13, C11 to C14, C12 to C15, C13 to C16, C1 to C17, C2 to C18, C3 to C19, C18 to C2, C4 to C20, C5 to C21, C6 to C22, C15 to C3, C19 to C4, C20 to C5, C21 to C6, C16 to C7, C22 to C8, C14 to C9, D6 to D1, D7 to D2, D8 to D3, D9 to D4, D4 to D5, D5 to D6, D1 to D7, D2 to D8, D3 to D9, J13 to J1, J8 to J10, J10 to J12, J11 to J13, J12 to J2, J1 to J3, J7 to J9, R31 to R1, R26 to R10, R27 to R11, R24 to R12, R21 to R13, R22 to R14, R23 to R15, R36 to R16, R2 to R17, R37 to R18, R4 to R19, R29 to R2, R38 to R20, R6 to R21, R39 to R22, R8 to R23, R40 to R24, R10 to R25, R11 to R26, R12 to R27, R13 to R28, R14 to R29, R32 to R3, R41 to R30, R16 to R31, R17 to R32, R18 to R33, R19 to R34, R20 to R35, R33 to R4, R34 to R5, R30 to R6, R28 to R7, R35 to R8, R25 to R9, RV5 to RV1, U6 to U10, U7 to U11, U11 to U2, U10 to U3, U9 to U5, U2 to U6, U3 to U7, U4 to U8, U5 to U9
Routing:
- net GND: track 410.6 -> 13.2 mm, vias 33 -> 6
- net +3.3V: track 220.2 -> 0.00 mm, vias 1 -> 0
- net /MicroController/MS2: track 135.5 -> 0.00 mm
- net /MicroController/STEP1: track 149.8 -> 15.8 mm
- net /MicroController/MS1: track 130.0 -> 0.00 mm
- net VDD: track 8.79 -> 126.9 mm
- net /MicroController/MS3: track 109.7 -> 0.00 mm
- net /MicroController/LED_F: track 39.2 -> 0.00 mm
- net /MicroController/LED_L: track 26.7 -> 0.00 mm
- net /MicroController/LED_B: track 26.2 -> 0.00 mm
- net Net-(J13-Pin_2): track 29.2 -> 2.98 mm
- net +BATT: track 254.7 -> 228.6 mm
- net /MicroController/ENABLE_B: track 27.9 -> 2.36 mm
- net /MicroController/ENABLE_L: track 24.8 -> 2.18 mm
- net /MicroController/LED_R: track 22.5 -> 0.00 mm
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
Commit message: feat: finish pcb design
Parts:
- added H1: MountingHole, MountingHole:MountingHole_3.2mm_M3, F.Cu at (96.9, 66.5)
- added H2: MountingHole, MountingHole:MountingHole_3.2mm_M3, F.Cu at (185.9, 66.5)
- added H3: MountingHole, MountingHole:MountingHole_3.2mm_M3, F.Cu at (185.9, 132.6)
- added H4: MountingHole, MountingHole:MountingHole_3.2mm_M3, F.Cu at (96.9, 132.6)
- added U4: LXDC55FAAA-203, mylib:LXDC55FAAA203, F.Cu at (112.2, 84.0)
- added Y1: XRCGB16M000FXN02R0, bldc_lib:XRCGB, F.Cu at (119.4, 88.7)
- J1: footprint Connector_PinSocket_2.54mm:PinSocket_1x04_P2.54mm_Horizontal -> Connector_PinSocket_2.54mm:PinSocket_1x04_P2.54mm_Vertical; moved to B.Cu
- R12: moved to B.Cu
- moved R8 43.9 mm to (109.8, 87.8)
- moved RV1 43.8 mm to (108.8, 94.8)
- moved C11 36.3 mm to (109.7, 83.1), turned to 90 degrees
- moved C12 30.2 mm to (119.2, 80.2), turned to 90 degrees
- moved C13 27.9 mm to (120.7, 80.2), turned to 90 degrees
- moved R12 22.6 mm to (113.8, 77.8)
- moved F1 8.06 mm to (116.7, 65.2), turned to 180 degrees
- moved C2 5.46 mm to (117.6, 88.6)
- moved C6 5.22 mm to (113.6, 102.8), turned to 180 degrees
- moved C3 5.14 mm to (100.2, 83.5)
- moved SW1 5.14 mm to (100.2, 86.1)
- moved C7 5.11 mm to (98.4, 88.7)
- moved R7 5.11 mm to (101.9, 88.6)
- moved SW2 5.11 mm to (100.2, 91.2)
- moved C1 5.05 mm to (119.5, 87.0)
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Connections:
- D7 pad 1: GND -> Net-(D7-K)
- D7 pad 2: Net-(D7-A) -> VDD
- J1 pad 2: /MicroController/SWCLK -> /MicroController/SWDIO
- J1 pad 3: /MicroController/SWDIO -> /MicroController/SWCLK
- R13 pad 1: VDD -> Net-(D7-K)
- R13 pad 2: Net-(D7-A) -> GND
- R15 pad 1: +3V3 -> +3.3V
- U2 pad 10: unconnected-(U2-PA2-Pad10) -> /MicroController/MS1
- U2 pad 11: unconnected-(U2-PA3-Pad11) -> /MicroController/MS2
- U2 pad 12: unconnected-(U2-PA4-Pad12) -> /MicroController/adc_speed
- U2 pad 13: unconnected-(U2-PA5-Pad13) -> /MicroController/MS3
- U2 pad 14: unconnected-(U2-PA6-Pad14) -> /MicroController/DIR_L
- U2 pad 15: unconnected-(U2-PA7-Pad15) -> /MicroController/DIR_U
- U2 pad 16: unconnected-(U2-PB0-Pad16) -> /MicroController/LED1
- U2 pad 17: unconnected-(U2-PB1-Pad17) -> /MicroController/LED2
- U2 pad 18: unconnected-(U2-PB2-Pad18) -> /MicroController/LED3
- U2 pad 2: unconnected-(U2-PC13-Pad2) -> /MicroController/ENABLE_U
- U2 pad 22: /MicroController/LED1 -> /MicroController/LED4
- U2 pad 25: unconnected-(U2-PB11-Pad25) -> /MicroController/LED_CAN_TX
- U2 pad 26: unconnected-(U2-PB12-Pad26) -> /MicroController/LED_CAN_RX
- U2 pad 27: unconnected-(U2-PB13-Pad27) -> /MicroController/DIR_D
- U2 pad 28: unconnected-(U2-PB14-Pad28) -> /MicroController/DIR_B
- U2 pad 29: unconnected-(U2-PB15-Pad29) -> /MicroController/STEP1
- U2 pad 3: unconnected-(U2-PC14-Pad3) -> /MicroController/ENABLE_R
- U2 pad 30: /MicroController/SW1 -> /MicroController/DIR_F
- U2 pad 31: /MicroController/LED_CAN_TX -> unconnected-(U2-PA9-Pad31)
- U2 pad 32: /MicroController/LED_CAN_RX -> unconnected-(U2-PA10-Pad32)
- U2 pad 39: unconnected-(U2-PA15-Pad39) -> /MicroController/LED_L
- U2 pad 4: unconnected-(U2-PC15-Pad4) -> /MicroController/ENABLE_L
- U2 pad 40: unconnected-(U2-PB3-Pad40) -> /MicroController/LED_B
- U2 pad 41: unconnected-(U2-PB4-Pad41) -> /MicroController/LED_R
- U2 pad 42: unconnected-(U2-PB5-Pad42) -> /MicroController/LED_F
- U2 pad 43: unconnected-(U2-PB6-Pad43) -> /MicroController/ENABLE_B
- U2 pad 44: unconnected-(U2-PB7-Pad44) -> /MicroController/ENABLE_F
- U2 pad 46: unconnected-(U2-PB9-Pad46) -> /MicroController/ENABLE_D
- U2 pad 8: unconnected-(U2-PA0-Pad8) -> /MicroController/SW1
- U2 pad 9: unconnected-(U2-PA1-Pad9) -> /MicroController/DIR_R
Routing:
- net +3.3V: track 0.00 -> 293.8 mm, vias 0 -> 5
- net /MicroController/MS3: track 0.00 -> 178.8 mm, vias 0 -> 3
- net /MicroController/MS2: track 0.00 -> 178.2 mm, vias 0 -> 3
- net /MicroController/MS1: track 0.00 -> 177.3 mm, vias 0 -> 2
- net /MicroController/STEP1: track 15.8 -> 169.5 mm, vias 0 -> 1
- net /MicroController/ENABLE_B: track 2.36 -> 80.0 mm
- net /MicroController/ENABLE_R: track 2.86 -> 80.3 mm, vias 0 -> 2
- net GND: track 13.2 -> 77.9 mm, vias 6 -> 487
- net /MicroController/DIR_R: track 0.00 -> 60.8 mm, vias 0 -> 2
- net /MicroController/ENABLE_D: track 2.49 -> 62.6 mm
- net +5V: track 0.00 -> 59.3 mm, vias 0 -> 3
- net /MicroController/NRST: track 0.00 -> 57.8 mm, vias 0 -> 1
- net /MicroController/ENABLE_L: track 2.18 -> 59.9 mm, vias 0 -> 2
- net /MicroController/DIR_B: track 0.00 -> 54.5 mm, vias 0 -> 2
- net /MicroController/ENABLE_F: track 2.05 -> 55.6 mm
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- added copper zone on F.Cu, net +3.3V
Other:
- outline, holes or cut-outs redrawn
- board text added: "3.3V"
- board text added: "5V"
- board text added: "CAL"
- board text added: "ERR"
- board text added: "RST"
- board text added: "RUN"
- board text added: "UI"
- board text added: "VM"

Commit message: fix: add UART
Parts:
- added J14: PH, Connector_JST:JST_PH_S2B-PH-K_1x02_P2.00mm_Horizontal, F.Cu at (100.9, 107.8)
- moved J2 6.96 mm to (100.9, 115.3)
- moved C9 6.96 mm to (107.7, 112.7)
- moved R9 6.96 mm to (104.1, 116.3)
- moved U3 6.96 mm to (109.3, 116.2)
- moved D5 4.12 mm to (111.1, 109.1)
- moved D6 4.12 mm to (111.1, 110.8)
- moved R11 4.12 mm to (107.8, 110.8)
- moved R10 4.12 mm to (107.8, 109.2)
Connections:
- U2 pad 31: unconnected-(U2-PA9-Pad31) -> /MicroController/USART_TX
- U2 pad 32: unconnected-(U2-PA10-Pad32) -> /MicroController/USART_RX
Routing:
- net /MicroController/USART_RX: track 0.00 -> 27.5 mm, vias 0 -> 1
- net /MicroController/USART_TX: track 0.00 -> 27.1 mm, vias 0 -> 1
- net +5V: track 59.3 -> 66.5 mm
- net /MicroController/CAN_TX: track 15.7 -> 22.7 mm
- net /MicroController/CAN_RX: track 15.0 -> 19.5 mm
- net /MicroController/SWDIO: track 41.1 -> 45.5 mm
- net /MicroController/LED_CAN_RX: track 15.4 -> 11.2 mm, vias 2 -> 0
- net /MicroController/LED_CAN_TX: track 13.4 -> 9.88 mm, vias 2 -> 0
- net /MicroController/SWCLK: track 43.5 -> 45.1 mm
- net /MicroController/DIR_F: track 22.8 -> 23.5 mm
- net GND: track 77.9 -> 78.3 mm, vias 487 -> 484
Other:
- board text added: "CAN"
- board text added: "ST-LINK"
- board text added: "UART"

Commit message: chore: add pdf
Parts:
- J14: footprint Connector_JST:JST_PH_S2B-PH-K_1x02_P2.00mm_Horizontal -> Connector_JST:JST_PH_S3B-PH-K_1x03_P2.00mm_Horizontal
- moved J2 1.56 mm to (100.8, 116.9)
- moved R9 1.56 mm to (104.0, 117.8)
Routing:
- net /MicroController/SWCLK: track 45.1 -> 46.6 mm
- net /MicroController/SWDIO: track 45.5 -> 44.5 mm
- net /MicroController/CAN_H: track 6.72 -> 7.52 mm
- net GND: track 78.3 -> 78.5 mm, vias 484 -> 489
